File: documentation/BertheVarioTac-Shema/BertheVarioTac-Shema.kicad_sch (KiCad schematic)
At the start: 1 part, among them P1 4P-1.25 Power supply base

Commit message: kicad shema
Parts:
- added CN1: 4P-1.25 Temperature and humidity interface, symbol Connector_Generic:Conn_01x04
- added P3: 4P-1.25 Extended IO, symbol Connector_Generic:Conn_01x04
- added RV10K: R_Potentiometer, symbol Device:R_Potentiometer
Connections:
- net GNDREF: now also RV10K.3
- new net: P3.3 (Pin_3), RV10K.2
- no-connect marks 0 -> 10
Other:
- note added: "+3.3V to Gps, BMP180 and HMC5883L"
- note added: "GND to VBat -"
- note added: "GPS Tx"
- note added: "IO22 to SCL BMP180"
- note added: "IO22 to SCL HMC5883L"
- note added: "IO27 to SDA BMP180"
- note added: "IO27 to SDA HMC5883L"
- note added: "IO35 to VBat +"
- note added: "to 5v Bat converter GND, GPS, BMP180 and HMC5883L"
- note added: "to 5v Bat converter VDD"
- moved on the sheet: P1

Commit message: mise a jour kicad
Parts:
- added BMP180, HMC5883L: ~, symbol BertheLibrary:I2C-COMPOSANT
- added BT1: Battery_Cell, symbol Device:Battery_Cell
- added ESP32-2432S: ~, symbol BertheLibrary:ESP32
- added GPS-NEO6M: ~, symbol BertheLibrary:GPS-NEO6
- added P4: 2P-1.25 SPEAK, symbol Connector_Generic:Conn_01x02
- added R1: R 100 ohms, symbol Device:R_Small
- added S1: Speaker, symbol Device:Speaker
- P1: renamed from RV10K; value R_Potentiometer -> Potentiometer 10k ohms
Connections:
- net GNDREF: now also GPS-NEO6M. (VCC)
- net at P1.2 (Pin_2): now also GPS-NEO6M. (VCC)
- net at CN1.1 (Pin_1): now also GPS-NEO6M. (VCC), HMC5883L. (VIN)
- net at CN1.2 (Pin_2): now also BMP180. (VIN), HMC5883L. (VIN)
- net at P3.2 (Pin_2): now also BMP180. (VIN), HMC5883L. (VIN)
- net at P3.4 (Pin_4): now also BT1.2 (-)
- net at P1.1: now also BT1.1 (+)
- new net: P4.1 (Pin_1), R1.1
- new net: R1.2, S1.2
- new net: P4.2 (Pin_2), S1.1
- no-connect marks 10 -> 9
Other:
- note added: "+3.3V to BMP180"
- note added: "IO22 SCL"
- note added: "IO27 SDA"
- note removed: "+3.3V to Gps, BMP180 and HMC5883L"
- note removed: "GPS Tx"
- note removed: "IO22 to SCL BMP180"
- note removed: "IO22 to SCL HMC5883L"
- note removed: "IO27 to SDA BMP180"
- note removed: "IO27 to SDA HMC5883L"
- moved on the sheet: CN1, P1, P3

Commit message: mise a jour kicad
Parts:
- added Lipo-1S-to-5V: ~, symbol BertheLibrary:Lipo-to-5v
- added SW1: SW_DIP_x01, symbol Switch:SW_DIP_x01
- added Usb-C-charger: ~, symbol BertheLibrary:Usb_c_charger
- S1: value Speaker -> Speaker 2W 8ohms
Connections:
- net GNDREF: now also Lipo-1S-to-5V. (OUT_5V)
- net VDD: now also SW1.1
- net at HMC5883L. (VIN): now also CN1.1 (Pin_1), GPS-NEO6M. (VCC)
- net at BT1.1 (+), P1.1: now also Lipo-1S-to-5V. (OUT_5V), Usb-C-charger. (B+)
- net at BT1.2 (-), P3.4 (Pin_4): now also Usb-C-charger. (B+)
- new net: BMP180. (VIN), CN1.2 (Pin_2), HMC5883L. (VIN)
- new net: BMP180. (VIN), HMC5883L. (VIN), P3.2 (Pin_2)
- new net: Lipo-1S-to-5V. (OUT_5V), SW1.2
- now unconnected: BMP180. (VIN), BMP180. (VIN)
- no-connect marks 9 -> 10
Other:
- note added: "3.3v"
- note added: "GND"
- moved on the sheet: BMP180, BT1, CN1, ESP32-2432S, GPS-NEO6M, HMC5883L, P1, P3, P4, R1, S1

Commit message: modification ihm
Parts:
- renumbered BMP180 to BMP180_Pres., ESP32-2432S to ESP32-2432S_WROOM-32, HMC5883L to HMC5883L_Mag.
Connections:
- net GNDREF: now also BT1.2 (-), Usb-C-charger. (B+)
- net at HMC5883L_Mag.. (VIN): now also CN1.1 (Pin_1), GPS-NEO6M. (VCC)
- net at BT1.1 (+), P1.1, Usb-C-charger. (B+): no longer Lipo-1S-to-5V. (OUT_5V)
- new net: BMP180_Pres.. (VIN), CN1.2 (Pin_2), HMC5883L_Mag.. (VIN)
- new net: BMP180_Pres.. (VIN), HMC5883L_Mag.. (VIN), P3.2 (Pin_2)
- now unconnected: BMP180_Pres.. (VIN), BMP180_Pres.. (VIN), P3.4 (Pin_4)
- no-connect marks 10 -> 5
Other:
- note added: "+3.3v"
- note added: "IO21"
- note added: "NC"
- note added: "Rx"
- note added: "Tx"
- note added: "VIN"
- note added: "to GND Battery converter, GPS, BMP180 and HMC5883L"
- note added: "to Vdd Out Battery converter"
- note removed: "to 5v Bat converter GND, GPS, BMP180 and HMC5883L"
- note removed: "to 5v Bat converter VDD"
- moved on the sheet: BT1, GPS-NEO6M

Commit message: modification kicad
Parts:
- renumbered ESP32-2432S_WROOM-32 to ESP32-2432S028_WROOM-32
Connections:
- net at HMC5883L_Mag.. (VIN): now also CN1.1 (Pin_1), GPS-NEO6M. (VCC)
- new net: BMP180_Pres.. (VIN), CN1.2 (Pin_2), HMC5883L_Mag.. (VIN)
- new net: BMP180_Pres.. (VIN), HMC5883L_Mag.. (VIN), P3.2 (Pin_2)
- now unconnected: BMP180_Pres.. (VIN), BMP180_Pres.. (VIN)
Changed lines of the file:
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@@
   (symbol (lib_id "BertheLibrary:ESP32") (at 86.36 62.23 0) (unit 1)
     (in_bom yes) (on_board yes) (dnp no)
-    (property "Reference" "ESP32-2432S_WROOM-32" (at 73.66 60.96 0)
+    (property "Reference" "ESP32-2432S028_WROOM-32" (at 73.66 60.96 0)
       (effects (font (size 1.27 1.27)) (justify left))
     )
@@
       (project "BertheVarioTac-Shema"
         (path "/20a72893-107a-4d28-9717-d104a5df1eab"
-          (reference "ESP32-2432S_WROOM-32") (unit 1)
+          (reference "ESP32-2432S028_WROOM-32") (unit 1)
         )
       )

Commit message: modification kicad
Connections:
- net VDD: now also Lipo-1S-to-5V. (OUT_5V); no longer SW1.1
- net at HMC5883L_Mag.. (VIN): now also CN1.1 (Pin_1), GPS-NEO6M. (VCC)
- net at SW1.2: now also BT1.1 (+), Usb-C-charger. (B+); no longer Lipo-1S-to-5V. (OUT_5V)
- new net: BMP180_Pres.. (VIN), CN1.2 (Pin_2), HMC5883L_Mag.. (VIN)
- new net: BMP180_Pres.. (VIN), HMC5883L_Mag.. (VIN), P3.2 (Pin_2)
- new net: Lipo-1S-to-5V. (OUT_5V), P1.1, SW1.1
- now unconnected: BMP180_Pres.. (VIN), BMP180_Pres.. (VIN)
Other:
- moved on the sheet: BMP180_Pres., BT1, CN1, ESP32-2432S028_WROOM-32, GPS-NEO6M, HMC5883L_Mag., Lipo-1S-to-5V, P1, P3, P4, R1, S1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
