File: documentation/06-BertheVarioTac-Shema/BertheVarioTac-Shema.kicad_pcb (KiCad board)
At the start: 2 copper layers, 15 parts, among them CN1 4P-1.25 Temperature and humid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, P1 4P-1.25 Power supply base, P3 4P-1.25 Extended IO, P4 2P-1.25 SPEAK, P5 10 k ohms, SW1 SW_DIP_x01

Commit message: modification pcb
Parts:
- added QMC5883_Mag1: ~, BertheShema:QMC5883, F.Cu at (102.9, 117.9)
- P1: value 4P-1.25 Power supply base -> Power supply base
- moved P3 67.6 mm to (111.8, 144.8), turned to 90 degrees
- moved P1 25.5 mm to (160.0, 144.8), turned to 90 degrees
- moved CN1 21.8 mm to (137.2, 144.8), turned to 90 degrees

Commit message: modification pcb
Parts:
- moved GPS-NEO6M1 19.0 mm to (123.0, 99.0)
- moved BMP180_Press.1 12.5 mm to (173.0, 130.5)
- moved Lipo-1S-to-5V1 10.5 mm to (168.0, 99.0)
- moved P1 7.02 mm to (164.0, 139.0)
- moved P3 6.79 mm to (111.5, 138.0)
- moved CN1 5.79 mm to (137.5, 139.0)
- moved QMC5883_Mag.1 5.78 mm to (107.0, 99.0)
Routing:
- net Net-(BMP180_Press.1-VCC): track 30.5 -> 0.00 mm
- net Net-(BMP180_Press.1-SCL): track 30.5 -> 0.00 mm
- net GNDREF: track 30.5 -> 0.00 mm
- net Net-(BMP180_Press.1-SDA): track 30.5 -> 39.6 mm
Other:
- board outline added: 86 x 50 mm
Changed lines of the file:
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@@
   )
   (footprint "BertheShema:4 trous standard" (layer "F.Cu")
-    (at 137.16 144.78 90)
+    (at 137.46 139 90)
     (property "Sheetfile" "BertheVarioTac-Shema.kicad_sch")
     (property "Sheetname" "")
@@
   )
   (footprint "BertheShema:4 trous standard" (layer "F.Cu")
-    (at 185.42 132.08)
+    (at 173 130.54)
     (property "Sheetfile" "BertheVarioTac-Shema.kicad_sch")
     (property "Sheetname" "")
@@
   )
   (footprint "BertheShema:4 trous standard" (layer "F.Cu")
-    (at 137.16 86.36)
+    (at 123 99)
     (property "Sheetfile" "BertheVarioTac-Shema.kicad_sch")
     (property "Sheetname" "")
@@
   )
   (footprint "BertheShema:3 trous standard" (layer "F.Cu")
-    (at 175.26 91.44)
+    (at 168 99)
     (property "Sheetfile" "BertheVarioTac-Shema.kicad_sch")
     (property "Sheetname" "")
@@
   )
   (footprint "BertheShema:4 trous standard" (layer "F.Cu")
-    (at 160.02 144.78 90)
+    (at 164 139 90)
     (property "Sheetfile" "BertheVarioTac-Shema.kicad_sch")
     (property "Sheetname" "")
@@
   )
   (footprint "BertheShema:4 trous standard" (layer "F.Cu")
-    (at 111.76 144.78 90)
+    (at 111.46 138 90)
     (property "Sheetfile" "BertheVarioTac-Shema.kicad_sch")
     (property "Sheetname" "")
@@
   )
   (footprint "BertheShema:4 trous standard" (layer "F.Cu")
-    (at 104.14 93.98)
+    (at 107 99)
     (property "Sheetfile" "BertheVarioTac-Shema.kicad_sch")
     (property "Sheetname" "")
@@
     (pad "4" thru_hole circle (at 0 -5.08) (size 1.8 1.8) (drill 0.8) (layers "*.Cu" "*.Mask"))
   )
-  (segment (start 185.42 134.62) (end 154.94 134.62) (width 0.2) (layer "B.Cu") (net 4))
-  (segment (start 185.42 127) (end 154.94 127) (width 0.2) (layer "B.Cu") (net 5))
-  (segment (start 185.42 132.08) (end 154.94 132.08) (width 0.2) (layer "B.Cu") (net 6))
-  (segment (start 185.42 129.54) (end 154.94 129.54) (width 0.2) (layer "B.Cu") (net 16))
+  (gr_arc (start 178 138) (mid 176.828427 140.828427) (end 174 142)
+    (stroke (width 0.05) (type default)) (layer "Edge.Cuts"))
+  (gr_circle (center 174 96) (end 175.6 96)
+    (stroke (width 0.05) (type default)) (fill none) (layer "Edge.Cuts"))
+  (gr_line (start 174 142) (end 96 142)
+    (stroke (width 0.05) (type default)) (layer "Edge.Cuts"))
+  (gr_line (start 96 92) (end 174 92)
+    (stroke (width 0.05) (type default)) (layer "Edge.Cuts"))
+  (gr_circle (center 96 138) (end 97.6 138)
+    (stroke (width 0.05) (type default)) (fill none) (layer "Edge.Cuts"))
+  (gr_arc (start 92 96) (mid 93.171573 93.171573) (end 96 92)
+    (stroke (width 0.05) (type default)) (layer "Edge.Cuts"))
+  (gr_arc (start 96 142) (mid 93.171573 140.828427) (end 92 138)
+    (stroke (width 0.05) (type default)) (layer "Edge.Cuts"))
+  (gr_line (start 92 138) (end 92 96)
+    (stroke (width 0.05) (type default)) (layer "Edge.Cuts"))
+  (gr_arc (start 174 92) (mid 176.828427 93.171573) (end 178 96)
+    (stroke (width 0.05) (type default)) (layer "Edge.Cuts"))
+  (gr_circle (center 96 96) (end 97.6 96)
+    (stroke (width 0.05) (type default)) (fill none) (layer "Edge.Cuts"))
+  (gr_circle (center 174 138) (end 175.6 138)
+    (stroke (width 0.05) (type default)) (fill none) (layer "Edge.Cuts"))
+  (gr_line (start 178 96) (end 178 138)
+    (stroke (width 0.05) (type default)) (layer "Edge.Cuts"))
+  (gr_line (start 96 92) (end 174 92)
+    (stroke (width 0.05) (type default)) (layer "B.CrtYd"))
+  (gr_arc (start 178 138) (mid 176.828427 140.828427) (end 174 142)
+    (stroke (width 0.05) (type default)) (layer "B.CrtYd"))
+  (gr_line (start 92 138) (end 92 96)
+    (stroke (width 0.05) (type default)) (layer "B.CrtYd"))
+  (gr_circle (center 174 138) (end 175.6 138)
+    (stroke (width 0.05) (type default)) (fill none) (layer "B.CrtYd"))
+  (gr_circle (center 174 96) (end 175.6 96)
+    (stroke (width 0.05) (type default)) (fill none) (layer "B.CrtYd"))
+  (gr_arc (start 174 92) (mid 176.828427 93.171573) (end 178 96)
+    (stroke (width 0.05) (type default)) (layer "B.CrtYd"))
+  (gr_arc (start 92 96) (mid 93.171573 93.171573) (end 96 92)
+    (stroke (width 0.05) (type default)) (layer "B.CrtYd"))
+  (gr_arc (start 96 142) (mid 93.171573 140.828427) (end 92 138)
+    (stroke (width 0.05) (type default)) (layer "B.CrtYd"))
+  (gr_line (start 178 96) (end 178 138)
+    (stroke (width 0.05) (type default)) (layer "B.CrtYd"))
+  (gr_line (start 174 142) (end 96 142)
+    (stroke (width 0.05) (type default)) (layer "B.CrtYd"))
+  (gr_circle (center 96 96) (end 97.6 96)
+    (stroke (width 0.05) (type default)) (fill none) (layer "B.CrtYd"))
+  (gr_circle (center 96 138) (end 97.6 138)
+    (stroke (width 0.05) (type default)) (fill none) (layer "B.CrtYd"))
+  (segment (start 129 135) (end 134 135) (width 0.2) (layer "B.Cu") (net 16))
+  (segment (start 134 135) (end 135 136) (width 0.2) (layer "B.Cu") (net 16))
+  (segment (start 104.394 121.666) (end 115.666 121.666) (width 0.2) (layer "B.Cu") (net 16))
+  (segment (start 135 136) (end 134.92 136.08) (width 0.2) (layer "B.Cu") (net 16))
+  (segment (start 115.666 121.666) (end 129 135) (width 0.2) (layer "B.Cu") (net 16))
+  (segment (start 134.92 136.08) (end 134.92 139) (width 0.2) (layer "B.Cu") (net 16))
+  (group "" (id 0c24f856-827c-4db5-bedc-1da90101af9d)
+    (members
+      0f9f0b0f-10d0-4955-aeab-e1cbe94f8aaf
+      1d9b28d2-06b9-404c-adb2-de31102f96a1
+      223a3170-5f80-4ce5-bbe9-b8b930264e48
+      26dfce0e-8679-4bfa-a42c-da5aa9b72e1e
+      33614b74-2ace-421b-9f19-22bc0e874804
+      429b46c1-531f-49cb-800f-b4dde87b6c70
+      4889d7a9-ad07-4583-91ea-aaed64f57fe2
+      6b1070e5-8a20-4791-b941-fc0960756bf0
+      826b8b91-82cd-45be-98eb-f7b463ab3d81
+      911cae65-0d15-454d-953d-11a9e9fa0e53
+      991e1e35-13ee-4674-b56a-04ca9e1af8ef
+      fd43a713-06b2-47a8-93d6-f73d757ec9dd
+    )
+  )
 )

Commit message: modification pcb
Parts:
- removed QMC5883_Mag.1: -, BertheShema:4 trous standard
- CN1: value 4P-1.25 Temperature and humidity interface -> Temperature and humidity interface
- GPS-NEO6M1: footprint BertheShema:4 trous standard -> BertheShema:GPSNEO6V2
- P3: value 4P-1.25 Extended IO -> Extended IO
- P4: value 2P-1.25 SPEAK -> SPEAK
- moved SW1 64.1 mm to (103.0, 140.0), turned to -90 degrees
- moved R1 52.3 mm to (107.0, 96.0)
- moved S1 51.8 mm to (119.0, 140.0), turned to 90 degrees
- moved P4 46.8 mm to (127.0, 140.0), turned to 90 degrees
- moved BT1 37.2 mm to (175.0, 108.0), turned to 180 degrees
- moved P3 26.2 mm to (137.5, 140.0)
- moved ESP32-2432S028_WROOM-32 26.1 mm to (135.0, 101.0)
- moved P5 25.2 mm to (107.0, 106.0), turned to 90 degrees
- moved GPS-NEO6M1 24.2 mm to (127.5, 122.8), turned to 90 degrees
- moved QMC5883_Mag1 15.8 mm to (92.5, 129.8)
- moved CN1 13.0 mm to (150.5, 140.0)
- moved Usb-C-charger1 9.49 mm to (156.0, 105.0)
- moved P1 1.00 mm to (164.0, 140.0)
Connections:
- GPS-NEO6M1 pad 1: (no net) -> GNDREF
- GPS-NEO6M1 pad 2: (no net) -> Net-(GPS-NEO6M1-TX)
- GPS-NEO6M1 pad 3: (no net) -> unconnected-(GPS-NEO6M1-RX-Pad3)
- GPS-NEO6M1 pad 4: (no net) -> Net-(BMP180_Press.1-VCC)
Routing:
- net Net-(BMP180_Press.1-SDA): track 39.6 -> 0.00 mm

Commit message: modification pcb
Parts:
- removed BMP180_Press.1: ~, BertheShema:4 trous standard
- added BMP180_Press1: ~, BertheShema:BMP180, F.Cu at (144.0, 124.0)
- Lipo-1S-to-5V1: footprint BertheShema:3 trous standard -> BertheShema:1S-to-5v
- Usb-C-charger1: footprint BertheShema:2 trous standard -> BertheShema:Usb-C-Charger
- moved SW1 71.8 mm to (174.0, 129.5), turned to 180 degrees
- moved R1 43.3 mm to (101.8, 139.0)
- moved BT1 25.3 mm to (167.0, 132.0)
- moved Lipo-1S-to-5V1 17.4 mm to (151.0, 102.5)
- moved Usb-C-charger1 13.2 mm to (169.0, 107.0), turned to -90 degrees
- moved P5 12.2 mm to (117.0, 99.0), turned to -90 degrees
- moved QMC5883_Mag1 4.48 mm to (88.9, 127.1)
Connections:
- CN1 pad 1: GNDREF -> Net-(BMP180_Press1-VIN)
- CN1 pad 2: Net-(BMP180_Press.1-SCL) -> Net-(BMP180_Press1-SDA)
- CN1 pad 3: Net-(BMP180_Press.1-SDA) -> Net-(BMP180_Press1-SCL)
- CN1 pad 4: Net-(BMP180_Press.1-VCC) -> GNDREF
- GPS-NEO6M1 pad 4: Net-(BMP180_Press.1-VCC) -> Net-(BMP180_Press1-VIN)
- Lipo-1S-to-5V1 pad 1: (no net) -> Net-(Lipo-1S-to-5V1-OUT_5V)
- Lipo-1S-to-5V1 pad 2: (no net) -> Net-(Lipo-1S-to-5V1-IN_3.7v)
- Lipo-1S-to-5V1 pad 3: (no net) -> GNDREF
- QMC5883_Mag1 pad 1: Net-(BMP180_Press.1-SDA) -> Net-(BMP180_Press1-VIN)
- QMC5883_Mag1 pad 2: Net-(BMP180_Press.1-SCL) -> GNDREF
- QMC5883_Mag1 pad 3: GNDREF -> Net-(BMP180_Press1-SCL)
- QMC5883_Mag1 pad 4: Net-(BMP180_Press.1-VCC) -> Net-(BMP180_Press1-SDA)
- Usb-C-charger1 pad 1: (no net) -> GNDREF
- Usb-C-charger1 pad 2: (no net) -> Net-(BT1-+)

Commit message: modification pcb
Parts:
- P5: footprint Potentiometer_THT:Potentiometer_ACP_CA14-H4_Horizontal -> BertheShema:potentiometre
- moved ESP32-2432S028_WROOM-32 19.7 mm to (152.0, 111.0)
- moved Lipo-1S-to-5V1 13.0 mm to (138.0, 102.5)
- moved SW1 7.65 mm to (167.0, 132.5), turned to 0 degrees
- moved Usb-C-charger1 6.00 mm to (175.0, 107.0)
- moved BT1 5.39 mm to (172.0, 130.0)
- moved BMP180_Press1 2.90 mm to (146.9, 124.0)
- moved P5 2.55 mm to (114.5, 99.5), turned to 0 degrees
- moved GPS-NEO6M1 1.26 mm to (128.4, 122.0)
Routing:
- net GNDREF: track 0.00 -> 198.4 mm
- net Net-(BMP180_Press1-VIN): track 0.00 -> 84.1 mm
- net Net-(BMP180_Press1-SCL): track 0.00 -> 79.3 mm
- net Net-(BMP180_Press1-SDA): track 0.00 -> 77.3 mm
- net Net-(Lipo-1S-to-5V1-IN_3.7v): track 0.00 -> 69.0 mm
- net Net-(GPS-NEO6M1-TX): track 0.00 -> 47.3 mm
- net Net-(Lipo-1S-to-5V1-OUT_5V): track 0.00 -> 47.2 mm
- net Net-(P3-Pin_3): track 0.00 -> 47.2 mm
- net Net-(BT1-+): track 0.00 -> 22.4 mm
- net Net-(R1-Pad1): track 0.00 -> 16.5 mm
- net Net-(P4-Pin_1): track 0.00 -> 16.2 mm
- net Net-(P4-Pin_2): track 0.00 -> 5.46 mm
