File: documentation/06-BertheVarioTac-Shema/BertheVarioTac-Shema.kicad_sch (KiCad schematic)
At the start: 15 parts, among them CN1 Temperature and humidity inte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, P1 Power supply base, P3 Extended IO, P4 SPEAK, P5 10 k ohms, SW1 SW_DIP_x01

Commit message: modification pcb
Parts:
- removed BMP180_Press.1: ~, BertheShema:4 trous standard, symbol BertheLibrary:carre_simple
- added BMP180_Press1: ~, BertheShema:BMP180, symbol BertheLibrary:BMP180
- Lipo-1S-to-5V1: footprint BertheShema:3 trous standard -> BertheShema:1S-to-5v
- Usb-C-charger1: footprint BertheShema:2 trous standard -> BertheShema:Usb-C-Charger
Connections:
- net GNDREF: now also CN1.4 (Pin_4), Lipo-1S-to-5V1.3 (GND), QMC5883_Mag1.2 (GND), Usb-C-charger1.1 (B-), BMP180_Press1.3 (GND); no longer CN1.1 (Pin_1), Lipo-1S-to-5V1. (OUT_5V), QMC5883_Mag1.3 (GND), Usb-C-charger1. (B+)
- net at QMC5883_Mag1.1 (VCC): now also CN1.1 (Pin_1), GPS-NEO6M1.4 (VCC), BMP180_Press1.4 (VIN); no longer CN1.3 (Pin_3)
- net at CN1.2 (Pin_2): now also QMC5883_Mag1.4 (SDA), BMP180_Press1.1 (SDA); no longer QMC5883_Mag1.2 (SCL)
- net at P1.1 (Pin_1): now also Lipo-1S-to-5V1.1 (OUT_5V); no longer Lipo-1S-to-5V1. (OUT_5V)
- net at P5.1, SW1.1: now also Lipo-1S-to-5V1.2 (IN_3.7v); no longer Lipo-1S-to-5V1. (OUT_5V)
- net at BT1.1 (+), SW1.2: now also Usb-C-charger1.2 (+); no longer Usb-C-charger1. (B+)
- new net: BMP180_Press1.2 (SCL), CN1.3 (Pin_3), QMC5883_Mag1.3 (SCL)
Other:
- moved on the sheet: CN1

Commit message: modification pcb
Parts:
- P5: footprint Potentiometer_THT:Potentiometer_ACP_CA14-H4_Horizontal -> BertheShema:potentiometre
Connections:
- no-connect marks 1 -> 0
Other:
- note removed: "to GND Battery converter, GPS, BMP180 and HMC5883L"
Changed lines of the file:
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@@
   (title_block
     (title "BertheVarioTac")
-    (date "2024-10-06")
-    (rev "1.0")
+    (date "2024-10-07")
+    (rev "1.1")
     (comment 1 "Author : SpinBerthe")
   )
@@
   (junction (at 168.91 78.74) (diameter 0) (color 0 0 0 0)
   )
-  (junction (at 95.25 119.38) (diameter 0) (color 0 0 0 0)
-  )
   (junction (at 140.97 111.76) (diameter 0) (color 0 0 0 0)
   )
@@
   (junction (at 196.85 20.32) (diameter 0) (color 0 0 0 0)
   )
-  (no_connect (at 99.06 119.38))
   (wire (pts (xy 236.22 152.4) (xy 236.22 158.75))
     (stroke (width 0) (type default))
@@
     (stroke (width 0) (type default))
   )
-  (wire (pts (xy 95.25 119.38) (xy 99.06 119.38))
-    (stroke (width 0) (type default))
-  )
   (wire (pts (xy 236.22 26.67) (xy 236.22 20.32))
     (stroke (width 0) (type default))
@@
     (stroke (width 0) (type default))
   )
-  (wire (pts (xy 95.25 110.49) (xy 95.25 119.38))
+  (wire (pts (xy 95.25 110.49) (xy 95.25 129.54))
     (stroke (width 0) (type default))
   )
@@
     (stroke (width 0) (type default))
   )
-  (wire (pts (xy 95.25 119.38) (xy 95.25 129.54))
-    (stroke (width 0) (type default))
-  )
   (wire (pts (xy 220.98 156.21) (xy 220.98 144.78))
     (stroke (width 0) (type default))
@@
   )
   (text "IO35 to VBat +" (at 144.78 48.26 0)
-    (effects (font (size 1.27 1.27)) (justify left bottom))
-  )
-  (text "to GND Battery converter,\nGPS, BMP180 and HMC5883L"
-    (at 101.6 120.65 0)
     (effects (font (size 1.27 1.27)) (justify left bottom))
   )
@@
   (symbol (lib_id "Connector_Generic:Conn_01x04") (at 123.19 78.74 180) (unit 1)
     (in_bom yes) (on_board yes) (dnp no)
-    (property "Reference" "CN1" (at 123.19 69.85 0)
+    (property "Reference" "CN1" (at 125.73 69.85 0)
       (effects (font (size 1.27 1.27)))
     )
@@
   (symbol (lib_id "Connector_Generic:Conn_01x04") (at 123.19 52.07 180) (unit 1)
     (in_bom yes) (on_board yes) (dnp no)
-    (property "Reference" "P3" (at 123.19 44.45 0)
+    (property "Reference" "P3" (at 125.73 43.18 0)
       (effects (font (size 1.27 1.27)))
     )
@@
       (effects (font (size 1.27 1.27)) (justify right))
     )
-    (property "Footprint" "Potentiometer_THT:Potentiometer_ACP_CA14-H4_Horizontal" (at 170.18 49.53 0)
-      (effects (font (size 1.27 1.27)) hide)
-    )
+    (property "Footprint" "BertheShema:potentiometre" (at 170.18 49.53 0)
+      (effects (font (size 1.27 1.27)) hide)
+    )
