File: documentation/06-kicad/BertheVarioTac-Shema.kicad_sch (KiCad schematic)
At the start: 15 parts, among them CN1 Temperature and humidity inte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, P1 Power supply base, P3 Extended IO, P4 SPEAK, P5 10 k ohms, SW1 SW_DIP_x01

Commit message: modif pcb
Connections:
- net GNDREF: now also Lipo-1S-to-5V1.1 (GND); no longer Lipo-1S-to-5V1.3 (GND)
- net at P1.1 (Pin_1): now also Lipo-1S-to-5V1.3 (OUT_5V); no longer Lipo-1S-to-5V1.1 (OUT_5V)
Changed lines of the file:
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@@
     (title "BertheVarioTac")
     (date "2024-10-07")
-    (rev "1.1")
+    (rev "1.2")
     (comment 1 "Author : SpinBerthe")
   )
@@
   (junction (at 196.85 20.32) (diameter 0) (color 0 0 0 0)
   )
-  (wire (pts (xy 236.22 152.4) (xy 236.22 158.75))
-    (stroke (width 0) (type default))
-  )
   (wire (pts (xy 170.18 44.45) (xy 196.85 44.45))
     (stroke (width 0) (type default))
@@
     (stroke (width 0) (type default))
   )
-  (wire (pts (xy 58.42 130.81) (xy 58.42 156.21))
-    (stroke (width 0) (type default))
-  )
   (wire (pts (xy 77.47 110.49) (xy 95.25 110.49))
     (stroke (width 0) (type default))
@@
     (stroke (width 0) (type default))
   )
+  (wire (pts (xy 237.49 133.35) (xy 237.49 144.78))
+    (stroke (width 0) (type default))
+  )
   (wire (pts (xy 140.97 111.76) (xy 140.97 142.24))
     (stroke (width 0) (type default))
@@
     (stroke (width 0) (type default))
   )
-  (wire (pts (xy 58.42 156.21) (xy 220.98 156.21))
-    (stroke (width 0) (type default))
-  )
   (wire (pts (xy 40.64 69.85) (xy 44.45 69.85))
     (stroke (width 0) (type default))
   )
-  (wire (pts (xy 220.98 156.21) (xy 220.98 144.78))
-    (stroke (width 0) (type default))
-  )
   (wire (pts (xy 196.85 27.94) (xy 196.85 29.21))
     (stroke (width 0) (type default))
@@
     (stroke (width 0) (type default))
   )
+  (wire (pts (xy 58.42 130.81) (xy 58.42 152.4))
+    (stroke (width 0) (type default))
+  )
   (wire (pts (xy 170.18 53.34) (xy 170.18 59.69))
     (stroke (width 0) (type default))
@@
     (stroke (width 0) (type default))
   )
-  (wire (pts (xy 220.98 144.78) (xy 237.49 144.78))
-    (stroke (width 0) (type default))
-  )
   (wire (pts (xy 168.91 76.2) (xy 168.91 78.74))
     (stroke (width 0) (type default))
@@
     (stroke (width 0) (type default))
   )
-  (wire (pts (xy 237.49 152.4) (xy 236.22 152.4))
+  (wire (pts (xy 58.42 152.4) (xy 237.49 152.4))
     (stroke (width 0) (type default))
   )
@@
     )
   )
-  (symbol (lib_id "power:GNDREF") (at 236.22 158.75 0) (unit 1)
+  (symbol (lib_id "power:GNDREF") (at 237.49 133.35 180) (unit 1)
     (in_bom yes) (on_board yes) (dnp no) (fields_autoplaced)
-    (property "Reference" "#PWR0102" (at 236.22 165.1 0)
-      (effects (font (size 1.27 1.27)) hide)
-    )
-    (property "Value" "GNDREF" (at 236.22 163.83 0)
-      (effects (font (size 1.27 1.27)))
-    )
-    (property "Footprint" "" (at 236.22 158.75 0)
-      (effects (font (size 1.27 1.27)) hide)
-    )
-    (property "Datasheet" "" (at 236.22 158.75 0)
-      (effects (font (size 1.27 1.27)) hide)
-    )
+    (property "Reference" "#PWR0102" (at 237.49 127 0)
+      (effects (font (size 1.27 1.27)) hide)
+    )
+    (property "Value" "GNDREF" (at 240.03 132.08 0)
+      (effects (font (size 1.27 1.27)) (justify right))
+    )
+    (property "Footprint" "" (at 237.49 133.35 0)
+      (effects (font (size 1.27 1.27)) hide)
+    )
+    (property "Datasheet" "" (at 237.49 133.35 0)
+      (effects (font (size 1.27 1.27)) hide)
+    )

Commit message: R sda scl pcb
Parts:
- added R2, R3: 4.7k, BertheShema:R_47, symbol Device:R
Connections:
- net at BMP180_Press1.4 (VIN), CN1.1 (Pin_1), GPS-NEO6M1.4 (VCC)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: now also R2.1, R3.1
- net at BMP180_Press1.2 (SCL), CN1.3 (Pin_3), QMC5883_Mag1.3 (SCL): now also R3.2
- net at BMP180_Press1.1 (SDA), CN1.2 (Pin_2), QMC5883_Mag1.4 (SDA): now also R2.2
