File: documentation/06-kicad/BertheVarioTac-Shema.kicad_pcb (KiCad board)
At the start: 2 copper layers, 86 x 50 mm, 17 parts, among them CN1 Temperature and humidity inte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, P1 Power supply base, P3 Extended IO, P4 SPEAK, P5 10 k ohms, SW1 SW_DIP_x01

Commit message: modification pcb
Parts:
- moved SW1 5.50 mm to (173.5, 132.5)
- moved BT1 5.00 mm to (168.0, 130.0)
Routing:
- net Net-(Lipo-1S-to-5V1-IN_3.7v): track 65.3 -> 72.2 mm
- net Net-(BT1-+): track 23.0 -> 23.5 mm
- net Net-(Lipo-1S-to-5V1-OUT_5V): vias 1 -> 0
