File: kicad-pcb/BertheVarioTac-Shema.kicad_sch (KiCad schematic)
At the start: 17 parts, among them CN1 Temperature and humidity inte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, P1 Power supply base, P3 Extended IO, P4 SPEAK, P5 10 k ohms, SW1 SW_DIP_x01

Commit message: modif pcb batterie
Parts:
- BT1: footprint BertheShema:2 trous standard -> BertheShema:batterie
Changed lines of the file:
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@@
       (effects (font (size 1.27 1.27)) (justify left))
     )
-    (property "Footprint" "BertheShema:2 trous standard" (at 196.85 24.384 90)
+    (property "Footprint" "BertheShema:batterie" (at 196.85 24.384 90)
       (effects (font (size 1.27 1.27)) hide)
     )
